File: in_out_conn.sch (KiCad schematic (older format))
At the start: 73 parts, among them J1 JACK_2P, SW1 SW_PUSH, SW2 SW_PUSH, U3 MAX202, U4 74HC125, U5 MAX202, U7 PCA82C251, U8 MAX202

Commit message: add some pin headers to the BOM
Parts:
- J1: JLC (none) -> DC-IN-TH_DC-005-20A; LCSC (none) -> C136744
- UARTCAN0: JLC (none) -> DB9-TH_ID09S33E4GV00LF; LCSC (none) -> C185657
Changed lines of the file:
@@
 F 2 "connect:JACK_ALIM" H 8750 5550 60  0001 C CNN
 F 3 "" H 8750 5550 60  0001 C CNN
+F 4 "DC-IN-TH_DC-005-20A" H 8750 5550 50  0001 C CNN "JLC"
+F 5 " C136744" H 8750 5550 50  0001 C CNN "LCSC"
 	1    8750 5550
 	1    0    0    -1
@@
 F 2 "connect:DB9FC" H 1050 2300 60  0001 C CNN
 F 3 "" H 1050 2300 60  0001 C CNN
+F 4 "DB9-TH_ID09S33E4GV00LF" H 1050 2300 50  0001 C CNN "JLC"
+F 5 "C185657" H 1050 2300 50  0001 C CNN "LCSC"
 	1    1050 2300
 	-1   0    0    1
