File: kit-dev-coldfire-xilinx_5213.sch (KiCad schematic (older format))
At the start: 68 parts, among them Q1 3906, U1 MCF5213-LQFP100, U2 74AHC1G14, Y1 8MHz

Commit message: add some pin headers to the BOM
Parts:
- CT1, VDDA1: JLC (none) -> HDR-TH_2P-P2.54-V; LCSC (none) -> C358684
Changed lines of the file:
@@
 F 2 "Connector_PinHeader_2.54mm:PinHeader_1x02_P2.54mm_Vertical" H 14200 4450 60  0001 C CNN
 F 3 "" H 14200 4450 60  0001 C CNN
+F 4 "HDR-TH_2P-P2.54-V" H 14200 4450 50  0001 C CNN "JLC"
+F 5 " C358684" H 14200 4450 50  0001 C CNN "LCSC"
 	1    14200 4450
 	1    0    0    -1
@@
 F 2 "Connector_PinHeader_2.54mm:PinHeader_1x02_P2.54mm_Vertical" H 1400 10000 60  0001 C CNN
 F 3 "" H 1400 10000 60  0001 C CNN
+F 4 "HDR-TH_2P-P2.54-V" H 1400 10000 50  0001 C CNN "JLC"
+F 5 "C358684" H 1400 10000 50  0001 C CNN "LCSC"
 	1    1400 10000
 	1    0    0    -1
