File: xilinx.sch (KiCad schematic (older format))
At the start: 21 parts, among them P1 CONN_6, P3 CONN_2X2, P4 CONN_20X2, U9 XCR3256-TQ144

Commit message: add some pin headers to the BOM
Parts:
- P1: JLC (none) -> HDR-TH_6P-P2.54-V; LCSC (none) -> C37208
Changed lines of the file:
@@
 F 2 "Connector_PinHeader_2.54mm:PinHeader_1x06_P2.54mm_Vertical" H 2350 1050 60  0001 C CNN
 F 3 "" H 2350 1050 60  0001 C CNN
+F 4 "HDR-TH_6P-P2.54-V" V 2350 1050 50  0001 C CNN "JLC"
+F 5 "C37208" V 2350 1050 50  0001 C CNN "LCSC"
 	1    2350 1050
 	-1   0    0    1
